File: pcb/sensor/rollino-sensor.kicad_sch (KiCad schematic)
At the start: 13 parts, among them J1 FH12-6S-0.5SH, U1 PMW3610DM-SUDU, U2 TPS7A0518PDBVR

Commit message: Route both PCBs, copper logo, 3D renders of the boards
pcb/gen/route.py has Freerouting route every net (edge and logo keep-outs,
retrying strategies until nothing is left unconnected) and pours GND;
pcb/gen/render_pcbs.sh renders both boards in Blender from KiCad's VRML,
with generated models for the upside-down XIAO and the PMW3610 + lens. The
ROLLINO logo is now bare copper on the back of the band instead of
silkscreen cut by the XIAO's cutout. Connector mounting tabs go to GND;
mounting holes have symbols; the band is 0.5 mm wider for the connectors'
escape routes.

Co-Authored-By: Claude Opus 5.5 <noreply@anthropic.com>
Parts:
- removed J1: FH12-6S-0.5SH, Connector_FFC-FPC:Hirose_FH12-6S-0.5SH_1x06-1MP_P0.50mm_Horizontal, symbol Connector_Generic:Conn_01x06
- added H1: M2, MountingHole:MountingHole_2.2mm_M2, symbol Mechanical:MountingHole
- added J1: FH12-6S-0.5SH, Connector_FFC-FPC:Hirose_FH12-6S-0.5SH_1x06-1MP_P0.50mm_Horizontal, symbol Connector_Generic_MountingPin:Conn_01x06_MountingPin
Connections:
- net +3V3: now also J1.1 (Pin_1)
- net GND: now also J1.2 (Pin_2), J1.MP (MountPin)
- net MOTION: now also J1.6 (Pin_6)
- net NCS: now also J1.5 (Pin_5)
- net SCLK: now also J1.3 (Pin_3)
- net SDIO: now also J1.4 (Pin_4)

Commit message: Shorter base band for a stock 50 mm FFC, parts list, FPC pin order fix
The base board's band now ends at about 110 degrees, with the FPC
connectors lying along it; each ribbon creases flat under its sensor pod
and runs along a channel in the case's underside, held by the cover.
The model solves the crease position from fpc_len = 50 (type B cable).
Connector pins are numbered from the ribbon's path so each signal meets
itself (the flipped sensor connector had reversed them).
Adds parts.md, the parts to order.

Co-Authored-By: Claude Opus 5.5 <noreply@anthropic.com>
Connections:
- net +3V3: now also J1.6 (Pin_6); no longer J1.1 (Pin_1)
- net GND: now also J1.5 (Pin_5); no longer J1.2 (Pin_2)
- net MOTION: now also J1.1 (Pin_1); no longer J1.6 (Pin_6)
- net NCS: now also J1.2 (Pin_2); no longer J1.5 (Pin_5)
- net SCLK: now also J1.4 (Pin_4); no longer J1.3 (Pin_3)
- net SDIO: now also J1.3 (Pin_3); no longer J1.4 (Pin_4)
Other:
- note added: "J1 (FPC): pins numbered so each signal meets itself through the ribbon (see pcb/readme.md)"
- note removed: "J1 (FPC): 1 +3V3, 2 GND, 3 SCLK, 4 SDIO, 5 NCS, 6 MOTION - same pinout as J1/J2 on the base board"

Commit message: Route the base board again, clear the antenna, sensor decoupling by the pins
The base board had come out with nothing routed to its FPC connectors:
Freerouting can't start a track from their pads at this angle. generate.py
now lays a stub out of each pad and route.py has Freerouting join those;
route.py only saves a board that is whole and that KiCad's DRC has nothing
to report on, trying its other strategies otherwise.

Base board: no pour by the XIAO's antenna (the strip between the notch and
the ball's hole), the supply laid across that strip on the back, each
connector's grounds with their own vias to the pours, the pours stitched
together. The bus moves to D4/D5 (the XIAO's only pins that aren't kept
for low frequencies), the right sensor's MOTION to D8, and the buttons are
left, middle, right on D0, D1, D9, so each side's lines stay on its side.

Sensor board: each capacitor by the pin it serves on a short wide track
(PixArt's rule for CP, CN and VCP), the regulator's output capacitor
against it, a ground rail with vias from pin 11, 1.8 V round the lens
cutout on the back, test pads for 1.8 V and GND. Same parts.

Firmware: the new pins, the sensors' angles as the case model has them
now (elevation -22), full transmit power. Case: a hole in the cover under
the XIAO's reset button. The XIAO's 3D model on the base board was a
mirror image.

Co-Authored-By: Claude Opus 5.5 <noreply@anthropic.com>
Parts:
- added TP1: +1V8, TestPoint:TestPoint_Pad_D1.0mm, symbol Connector:TestPoint
- added TP2: GND, TestPoint:TestPoint_Pad_D1.0mm, symbol Connector:TestPoint
Connections:
- net +1V8: now also TP1.1
- net GND: now also TP2.1
